File: PsU/New Project/AC_DC_AC/AC_DC_AC.kicad_sch (KiCad schematic)
At the start: 19 parts, among them T1 Transformer_1P_2S

Commit message: AC_DC_HVDC
Parts:
- removed C1: Capacitor_NP, Capacitor_THT:C_Disc_D3.0mm_W2.0mm_P2.50mm, symbol PCM_SL_Devices:Capacitor_NP
- removed C2: C_Rect_L19.0mm_W5.0mm_P15.00mm, Capacitor_THT_AKL:C_Rect_L19.0mm_W5.0mm_P15.00mm_MKS4, symbol PCM_Capacitor_AKL:C_Rect_L19.0mm_W5.0mm_P15.00mm
- removed C3, C4: C, symbol Device:C
- removed D1, D2, D3, D4, D5, D6, D7: 1N4007, Diode_THT:D_DO-41_SOD81_P10.16mm_Horizontal, symbol Diode:1N4007
- removed D10, D9: LED, symbol Device:LED
- removed R1, R2, R3, R4: R, symbol Device:R
- removed T1: Transformer_1P_2S, symbol Device:Transformer_1P_2S
- added C5, C7, C8: Capacitor_NP, Capacitor_THT:C_Disc_D3.0mm_W2.0mm_P2.50mm, symbol PCM_SL_Devices:Capacitor_NP
- added C6: Capacitor_PO, Capacitor_THT:CP_Radial_D5.0mm_P2.50mm, symbol PCM_SL_Devices:Capacitor_PO
- added D11, D12, D13, D14, D16, D17, D18: 1N4007, Diode_THT:D_DO-41_SOD81_P10.16mm_Horizontal, symbol Diode:1N4007
- added D15, D8: LED, symbol Device:LED
- added Q1: 2N5192, Package_TO_SOT_THT_AKL:TO-126-3_Vertical_ECB, symbol PCM_Transistor_BJT_AKL:2N5192
- added R5, R6, R7, R8: R, symbol Device:R
- added SW1: SW_SPDT, openinput:SW_Micro_Switch, symbol PCM_openinput:SW_SPDT
- added SW2: SW_DPST_x2, symbol Switch:SW_DPST_x2
- added T2: Transformer_1P_2S, symbol Device:Transformer_1P_2S
Connections:
- net at BT1.1 (+): now also D11.2 (A), D12.2 (A), SW2.1 (A)
- net at BT1.2 (-): now also D13.1 (K), D14.1 (K), R8.1
- new net: C5.1, C6.1, C7.1, D17.1 (K), D17.2 (A)
- new net: C6.2, D16.2 (A)
- new net: C5.2, D16.1 (K), D18.2 (A)
- new net: C7.2, D18.1 (K), Q1.3 (B), T2.3 (SA), T2.4 (SB)
- new net: D15.1 (K), Q1.2 (C), SW1.1 (C), T2.5 (SC)
- new net: SW1.2 (NO), SW1.3 (NC), SW2.2 (B)
- new net: R7.1, T2.6 (SD)
- new net: D15.2 (A), R8.2
- new net: C8.1, D8.2 (A)
- new net: D8.1 (K), R6.2
- new net VAC: C8.2, D11.1 (K), D12.1 (K), D13.2 (A), D14.2 (A), Q1.1 (E), R5.1, R5.2, R6.1, R7.2
